Commit message: feat: update params and launch file

File: install/robotics_class/share/robotics_class/urdf/depth_camera.urdf.xacro (robot description, xacro)
@@ -1,66 +1 @@
-<?xml version="1.0" encoding="utf-8"?>
-<robot name="depth_camera" xmlns:xacro="http://ros.org/wiki/xacro" >
-  <xacro:property name="M_PI"   value="3.1415926535897931"/>
-  <link
-    name="depth_cam_link">
-    <inertial>
-      <origin
-        xyz="0.000254340878565573 0.00268031633059271 -0.00569075323067275"
-        rpy="0 0 0" />
-      <mass
-        value="0.227980406655671" />
-      <inertia
-        ixx="4.8473190489023E-05"
-        ixy="8.29314946303069E-09"
-        ixz="-5.0952649884666E-09"
-        iyy="0.000408820027771005"
-        iyz="-1.36580074559918E-07"
-        izz="0.000429553467348926" />
-    </inertial>
-    <visual>
-      <origin
-        xyz="0 0 0"
-        rpy="0 0 1.57" />
-      <geometry>
-        <mesh
-          filename="package://robotics_class/models/jetauto/depth_camera_link.stl" />
-      </geometry>
-      <material name="black"/>
-    </visual>
-    <collision>
-      <origin
-        xyz="0 0 0"
-        rpy="0 0 1.57" />
-      <geometry>
-        <mesh
-          filename="package://robotics_class/models/jetauto/depth_camera_link_collision.stl" />
-      </geometry>
-    </collision>
-  </link>
-  <joint
-    name="joint1"
-    type="revolute">
-    <origin
-      xyz="0.0288581470059471 0 0.202093286991617"
-      rpy="-0.000131510931722419 0 0" />
-    <parent
-      link="base_link" />
-    <child
-      link="depth_cam_link" />
-    <axis
-      xyz="0 0 1" />
-    <limit
-      lower="-2.09"
-      upper="2.09"
-      effort="1000"
-      velocity="10" />
-  </joint>
-  <link name="depth_cam_frame" />
-  <joint
-    name="depth_cam_joint_sim"
-    type="fixed">
-    <origin xyz="0 0 0" rpy="${-M_PI/2} 0 ${-M_PI/2}" />
-    <parent link="depth_cam_link" />
-    <child link="depth_cam_frame" />
-  </joint>
-</robot>
+/home/jose/Documents/robotica/src/robotics_class/urdf/depth_camera.urdf.xacro

File: install/robotics_class/share/robotics_class/urdf/imu.urdf.xacro (robot description, xacro)
@@ -1,35 +1 @@
-<?xml version="1.0" encoding="utf-8"?>
-<robot name="imu" xmlns:xacro="http://ros.org/wiki/xacro">
-  <xacro:property name="M_PI" value="3.1415926535897931"/>
-  <link name="imu_link"/>
-  <joint
-    name="imu_joint"
-    type="fixed">
-    <origin
-      xyz="0 0 ${0.025 - 0.0295 + 0.0965/2 + 0.0678410821576746}"
-      rpy="0 0 0" />
-    <parent
-      link="base_link"/>
-    <child
-      link="imu_link"/>
-  </joint>
-  <gazebo reference="imu_link">
-    <gravity>true</gravity>
-    <sensor name="imu" type="imu">
-      <always_on>true</always_on>
-      <update_rate>100</update_rate>
-      <visualize>true</visualize>
-      <plugin name="gazebo_ros_imu_sensor" filename="libgazebo_ros_imu_sensor.so">
-        <ros>
-          <remapping>~/out:=/jetauto/imu/data</remapping>
-        </ros>
-        <body_name>imu_link</body_name>
-        <gaussian_noise>0.0</gaussian_noise>
-        <xyz_offset>0 0 0</xyz_offset>
-        <rpy_offset>0 0 0</rpy_offset>
-        <frame_name>imu_link</frame_name>
-        <initial_orientation_as_reference>false</initial_orientation_as_reference>
-      </plugin>
-    </sensor>
-  </gazebo>
-</robot>
+/home/jose/Documents/robotica/src/robotics_class/urdf/imu.urdf.xacro

File: install/robotics_class/share/robotics_class/urdf/inertial_matrix.xacro (robot description, xacro)
@@ -1,41 +1 @@
-<?xml version="1.0" encoding="utf-8"?>
-<robot name="jetauto" xmlns:xacro="http://ros.org/wiki/xacro">
-  <xacro:property name="M_PI" value="3.1415926535897931" />
-  <!-- Macro for inertia matrix -->
-  <xacro:macro name="sphere_inertial" params="m r">
-    <inertial>
-      <mass value="${m}" />
-      <inertia
-        ixx="${2*m*r*r/5}"
-        ixy="0"
-        ixz="0"
-        iyy="${2*m*r*r/5}"
-        iyz="0"
-        izz="${2*m*r*r/5}" />
-    </inertial>
-  </xacro:macro>
-  <xacro:macro name="cylinder_inertial" params="m r h">
-    <inertial>
-      <mass value="${m}" />
-      <inertia
-        ixx="${m*(3*r*r+h*h)/12}"
-        ixy = "0"
-        ixz = "0"
-        iyy="${m*(3*r*r+h*h)/12}"
-        iyz = "0"
-        izz="${m*r*r/2}" />
-    </inertial>
-  </xacro:macro>
-  <xacro:macro name="box_inertial" params="m w h d">
-    <inertial>
-      <mass value="${m}" />
-      <inertia
-        ixx="${m*(h*h+d*d)/12}"
-        ixy = "0"
-        ixz = "0"
-        iyy="${m*(w*w+d*d)/12}"
-        iyz = "0"
-        izz="${m*(w*w+h*h)/12}" />
-    </inertial>
-  </xacro:macro>
-</robot>
+/home/jose/Documents/robotica/src/robotics_class/urdf/inertial_matrix.xacro

File: install/robotics_class/share/robotics_class/urdf/jetauto.xacro (robot description, xacro)
@@ -1,9 +1 @@
-<?xml version="1.0" encoding="utf-8"?>
-<robot name="jetauto" xmlns:xacro="http://ros.org/wiki/xacro">
-    <xacro:include filename="$(find robotics_class)/urdf/materials.xacro"/>
-    <xacro:include filename="$(find robotics_class)/urdf/inertial_matrix.xacro" />
-    <xacro:include filename="$(find robotics_class)/urdf/imu.urdf.xacro"/>
-    <xacro:include filename="$(find robotics_class)/urdf/lidar.urdf.xacro"/>
-    <!-- <xacro:include filename="$(find robotics_class)/urdf/depth_camera.urdf.xacro"/> -->
-    <xacro:include filename="$(find robotics_class)/urdf/jetauto_car.urdf.xacro"/>
-</robot>
+/home/jose/Documents/robotica/src/robotics_class/urdf/jetauto.xacro

File: install/robotics_class/share/robotics_class/urdf/jetauto_car.urdf.xacro (robot description, xacro)
@@ -1,384 +1 @@
-<?xml version="1.0" encoding="utf-8"?>
-<robot name="jetauto" xmlns:xacro="http://ros.org/wiki/xacro" >
-  <xacro:property name="M_PI"               value="3.1415926535897931"/>
-  <xacro:property name="base_link_mass"     value="1.6" />
-  <xacro:property name="base_link_w"        value="0.297"/>
-  <xacro:property name="base_link_h"        value="0.145"/>
-  <xacro:property name="base_link_d"        value="0.11255"/>
-  <xacro:property name="wheel_link_mass"    value="0.1" />
-  <xacro:property name="wheel_link_radius"  value="0.049"/>
-  <xacro:property name="wheel_link_length"  value="0.04167"/>
-  <xacro:include filename="$(find robotics_class)/urdf/p3d_plugin.gazebo.xacro"/>
-  <link name="base_footprint"/>
-  <joint name="base_joint" type="fixed">
-    <parent link="base_link"/>
-    <child link="base_footprint"/>
-    <origin xyz="0.0 0.0 0.005" rpy="0 0 0"/>
-  </joint>
-  <link
-    name="base_link">
-    <xacro:box_inertial m="${base_link_mass}" w="${base_link_w}" h="${base_link_h}" d="${base_link_d}"/>
-    <visual>
-      <origin
-        xyz="0 0 0"
-        rpy="0 0 0" />
-      <geometry>
-        <mesh
-          filename="package://robotics_class/models/jetauto/base_link.stl" />
-      </geometry>
-      <material name="green"/>
-    </visual>
-    <collision>
-      <origin
-        xyz="${base_link_w/2.0 - 0.14810} 0 ${0.126437/2 + 0.02362364}"
-        rpy="0 0 0" />
-      <geometry>
-        <box size="${base_link_w} ${base_link_h} ${base_link_d}" />
-      </geometry>
-    </collision>
-  </link>
-  <link
-    name="back_shell_link">
-    <inertial>
-      <origin
-        xyz="-1.22838595456587E-05 0.00218574826309681 -0.0500522861933898"
-        rpy="0 0 0" />
-      <mass
-        value="0.0663478534899862" />
-      <inertia
-        ixx="5.65277934912267E-05"
-        ixy="-5.13394387877366E-11"
-        ixz="-4.07561372273553E-11"
-        iyy="4.33740893441632E-05"
-        iyz="-5.43059341238134E-06"
-        izz="6.86642544694324E-05" />
-    </inertial>
-    <visual>
-      <origin
-        xyz="0 0 0"
-        rpy="0 0 0" />
-      <geometry>
-        <mesh
-          filename="package://robotics_class/models/jetauto/back_shell_link.stl" />
-      </geometry>
-      <material name="black">
-      </material>
-    </visual>
-    <!--<collision>-->
-      <!--<origin-->
-        <!--xyz="0 0 0"-->
-        <!--rpy="0 0 0" />-->
-      <!--<geometry>-->
-        <!--<mesh-->
-          <!--filename="package://robotics_class/models/jetauto/back_shell_link.stl" />-->
-      <!--</geometry>-->
-    <!--</collision>-->
-  </link>
-  <joint
-    name="back_shell_joint"
-    type="fixed">
-    <origin
-      xyz="-0.076481 0 0.082796"
-      rpy="-3.1416 0 1.5708" />
-    <parent
-      link="base_link" />
-    <child
-      link="back_shell_link" />
-    <axis
-      xyz="0 0 0" />
-  </joint>
-  <link
-    name="wheel_right_front_link">
-    <xacro:cylinder_inertial m="${wheel_link_mass}" r="${wheel_link_radius}" h="${wheel_link_length}" />
-    <visual>
-      <origin
-        xyz="0 0 -0.004"
-        rpy="${M_PI} 0 0" />
-      <geometry>
-        <mesh
-          filename="package://robotics_class/models/jetauto/wheel_right_front_link.stl" />
-      </geometry>
-      <material name="black"/>
-    </visual>
-    <collision>
-      <origin
-        xyz="0 0 -0.025"
-        rpy="0 0 0" />
-      <geometry>
-        <cylinder length="${wheel_link_length}" radius="${wheel_link_radius}"/>
-        <!-- <sphere radius="${wheel_link_radius}"/> -->
-      </geometry>
-    </collision>
-  </link>
-  <joint
-    name="wheel_right_front_joint"
-    type="continuous">
-    <origin
-      xyz="0.097397 -0.086125 0.04508"
-      rpy="-1.5708 1.5708 0" />
-    <parent
-      link="base_link" />
-    <child
-      link="wheel_right_front_link" />
-    <axis
-      xyz="0 0 1"/>
-  </joint>
-  <link
-    name="wheel_left_front_link">
-    <xacro:cylinder_inertial m="${wheel_link_mass}" r="${wheel_link_radius}" h="${wheel_link_length}" />
-    <visual>
-      <origin
-        xyz="0 0 0.004"
-        rpy="${M_PI} 0 0" />
-      <geometry>
-        <mesh
-          filename="package://robotics_class/models/jetauto/wheel_left_front_link.stl" />
-      </geometry>
-      <material name="black"/>
-    </visual>
-    <collision>
-      <origin
-        xyz="0 0 0.025"
-        rpy="0 0 0" />
-      <geometry>
-        <cylinder length="${wheel_link_length}" radius="${wheel_link_radius}"/>
-        <!-- <sphere radius="${wheel_link_radius}"/> -->
-      </geometry>
-    </collision>
-  </link>
-  <joint
-    name="wheel_left_front_joint"
-    type="continuous">
-    <origin
-      xyz="0.097397 0.086125 0.04508"
-      rpy="-1.5708 1.5708 0" />
-    <parent
-      link="base_link" />
-    <child
-      link="wheel_left_front_link" />
-    <axis
-      xyz="0 0 1"/>
-  </joint>
-  <link
-    name="wheel_right_back_link">
-    <xacro:cylinder_inertial m="${wheel_link_mass}" r="${wheel_link_radius}" h="${wheel_link_length}" />
-    <visual>
-      <origin
-        xyz="0 0 -0.004"
-        rpy="${M_PI} 0 0" />
-      <geometry>
-        <mesh
-          filename="package://robotics_class/models/jetauto/wheel_right_back_link.stl" />
-      </geometry>
-      <material name="black"/>
-    </visual>
-    <collision>
-      <origin
-        xyz="0 0 -0.025"
-        rpy="0 0 0" />
-      <geometry>
-        <cylinder length="${wheel_link_length}" radius="${wheel_link_radius}"/>
-        <!-- <sphere radius="${wheel_link_radius}"/> -->
-      </geometry>
-    </collision>
-  </link>
-  <joint
-    name="wheel_right_back_joint"
-    type="continuous">
-    <origin
-      xyz="-0.097397 -0.086125 0.04508"
-      rpy="-1.5708 1.5708 0" />
-    <parent
-      link="base_link" />
-    <child
-      link="wheel_right_back_link" />
-    <axis
-      xyz="0 0 1"/>
-  </joint>
-  <link
-    name="wheel_left_back_link">
-    <xacro:cylinder_inertial m="${wheel_link_mass}" r="${wheel_link_radius}" h="${wheel_link_length}" />
-    <visual>
-      <origin
-        xyz="0 0 0.004"
-        rpy="${M_PI} 0 0" />
-      <geometry>
-        <mesh
-          filename="package://robotics_class/models/jetauto/wheel_left_back_link.stl" />
-      </geometry>
-      <material name="black"/>
-    </visual>
-    <collision>
-      <origin
-        xyz="0 0 0.025"
-        rpy="0 0 0" />
-      <geometry>
-        <!-- <sphere radius="${wheel_link_radius}"/> -->
-        <cylinder length="${wheel_link_length}" radius="${wheel_link_radius}"/>
-      </geometry>
-    </collision>
-  </link>
-  <joint
-    name="wheel_left_back_joint"
-    type="continuous">
-    <origin
-      xyz="-0.097397 0.086125 0.04508"
-      rpy="-1.5708 1.5708 0" />
-    <parent
-      link="base_link" />
-    <child
-      link="wheel_left_back_link" />
-    <axis
-      xyz="0 0 1"/>
-  </joint>
-  <gazebo reference="wheel_left_back_link">
-    <kp>5000000.0</kp>
-    <kd>100.0</kd>
-    <mu1>1.0</mu1>
-    <mu2>1.0</mu2>
-    <maxVel>1.0</maxVel>
-    <minDepth>0.002</minDepth>
-  </gazebo>
-  <gazebo reference="wheel_left_front_link">
-    <kp>5000000.0</kp>
-    <kd>100.0</kd>
-    <mu1>1.0</mu1>
-    <mu2>1.0</mu2>
-    <maxVel>1.0</maxVel>
-    <minDepth>0.002</minDepth>
-  </gazebo>
-  <gazebo reference="wheel_right_back_link">
-    <kp>5000000.0</kp>
-    <kd>100.0</kd>
-    <mu1>1.0</mu1>
-    <mu2>1.0</mu2>
-    <maxVel>1.0</maxVel>
-    <minDepth>0.002</minDepth>
-  </gazebo>
-  <gazebo reference="wheel_right_front_link">
-    <kp>5000000.0</kp>
-    <kd>100.0</kd>
-    <mu1>1.0</mu1>
-    <mu2>1.0</mu2>
-    <maxVel>1.0</maxVel>
-    <minDepth>0.002</minDepth>
-  </gazebo>
-  <xacro:p3d_plugin_macro
-    parent="base_link"
-    update_rate="100"
-    topic_name="odometry/ground_truth"
-    mass="0.00001"
-    body_name="base_link"
-    frame_name="base_footprint"
-    noise="0"
-    xyz_offset="0 0 0"
-    rpy_offset="0 0 0">
-    <inertia ixx="0.00001" ixy="0" ixz="0" iyy="0.00001" iyz="0" izz="0.00001"/>
-    <origin xyz="0 0 0" rpy="0 0 0"/>
-  </xacro:p3d_plugin_macro>
-  <gazebo>
-    <plugin name="gazebo_ros_planar_move" filename="libgazebo_ros_planar_move.so">
-      <ros>
-        <remapping>cmd_vel:=/jetauto/cmd_vel</remapping>
-        <remapping>odom:=/jetauto/odometry/unfiltered</remapping>
-      </ros>
-      <command_topic>/jetauto/cmd_vel</command_topic>
-      <odometry_topic>/jetauto/odometry/unfiltered</odometry_topic>
-      <odometry_frame>odom</odometry_frame>
-      <odometry_rate>100.0</odometry_rate>
-      <robot_base_frame>base_link</robot_base_frame>
-      <publish_odom>true</publish_odom>
-      <ground_truth>true</ground_truth>
-      <publish_odom_tf>true</publish_odom_tf>
-    </plugin>
-    <!-- <plugin name="gazebo_ros_diff_drive_back" filename="libgazebo_ros_diff_drive.so"> -->
-    <!--   <ros> -->
-    <!--     <remapping>odom:=jetauto/odometry/unfiltered</remapping> -->
-    <!--     <remapping>cmd_vel:=jetauto/cmd_vel</remapping> -->
-    <!--   </ros> -->
-    <!--   <!-1- Plugin update rate in Hz -1-> -->
-    <!--   <updateRate>100</updateRate> -->
-    <!--     <!-1- Name of left joint, defaults to `left_joint` -1-> -->
-    <!--   <left_joint>wheel_left_back_joint</left_joint> -->
-    <!--     <!-1- Name of right joint, defaults to `right_joint` -1-> -->
-    <!--   <right_joint>wheel_right_back_joint</right_joint> -->
-    <!--     <!-1- The distance from the center of one wheel to the other, in meters, defaults to 0.34 m -1-> -->
-    <!--   <wheel_separation>0.18</wheel_separation> -->
-    <!--     <!-1- Diameter of the wheels, in meters, defaults to 0.15 m -1-> -->
-    <!--   <wheel_diameter>0.098</wheel_diameter> -->
-    <!--     <!-1- Wheel acceleration, in rad/s^2, defaults to 0.0 rad/s^2 -1-> -->
-    <!--   <wheel_acceleration>1.0</wheel_acceleration> -->
-    <!--     <!-1- Maximum torque which the wheels can produce, in Nm, defaults to 5 Nm -1-> -->
-    <!--   <wheel_torque>5</wheel_torque> -->
-    <!--     <!-1- Topic to receive geometry_msgs/Twist message commands, defaults to `cmd_vel` -1-> -->
-    <!--   <command_topic>/jetauto/cmd_vel</command_topic> -->
-    <!--     <!-1- Topic to publish nav_msgs/Odometry messages, defaults to `odom` -1-> -->
-    <!--   <odometry_topic>jetauto/odom/unfiltered</odometry_topic> -->
-    <!--     <!-1- Odometry frame, defaults to `odom` -1-> -->
-    <!--   <odometry_frame>odom</odometry_frame> -->
-    <!--     <!-1- Robot frame to calculate odometry from, defaults to `base_footprint` -1-> -->
-    <!--   <robot_base_frame>base_footprint</robot_base_frame> -->
-    <!--     <!-1- Odometry source, 0 for ENCODER, 1 for WORLD, defaults to WORLD -1-> -->
-    <!--   <odometry_source>0</odometry_source> -->
-    <!--     <!-1- Set to true to publish transforms for the wheel links, defaults to false -1-> -->
-    <!--   <publish_wheel_tF>false</publish_wheel_tF> -->
-    <!--     <!-1- Set to true to publish transforms for the odometry, defaults to true -1-> -->
-    <!--   <publish_odom>true</publish_odom> -->
-    <!--     <!-1- Set to true to publish sensor_msgs/JointState on /joint_states for the wheel joints, defaults to false -1-> -->
-    <!--   <publish_wheel_joint_state>false</publish_wheel_joint_state> -->
-    <!--     <!-1- Set to true to swap right and left wheels, defaults to true -1-> -->
-    <!--   <legacy_mode>false</legacy_mode> -->
-    <!-- </plugin> -->
-    <!-- <plugin name="gazebo_ros_diff_drive_front" filename="libgazebo_ros_diff_drive.so"> -->
-    <!--   <ros> -->
-    <!--     <remapping>cmd_vel:=jetauto/cmd_vel</remapping> -->
-    <!--   </ros> -->
-    <!--   <!-1- Plugin update rate in Hz -1-> -->
-    <!--   <updateRate>100</updateRate> -->
-    <!--     <!-1- Name of left joint, defaults to `left_joint` -1-> -->
-    <!--   <left_joint>wheel_left_front_joint</left_joint> -->
-    <!--     <!-1- Name of right joint, defaults to `right_joint` -1-> -->
-    <!--   <right_joint>wheel_right_front_joint</right_joint> -->
-    <!--     <!-1- The distance from the center of one wheel to the other, in meters, defaults to 0.34 m -1-> -->
-    <!--   <wheel_separation>0.18</wheel_separation> -->
-    <!--     <!-1- Diameter of the wheels, in meters, defaults to 0.15 m -1-> -->
-    <!--   <wheel_diameter>0.098</wheel_diameter> -->
-    <!--     <!-1- Wheel acceleration, in rad/s^2, defaults to 0.0 rad/s^2 -1-> -->
-    <!--   <wheel_acceleration>1.0</wheel_acceleration> -->
-    <!--     <!-1- Maximum torque which the wheels can produce, in Nm, defaults to 5 Nm -1-> -->
-    <!--   <wheel_torque>5</wheel_torque> -->
-    <!--     <!-1- Topic to receive geometry_msgs/Twist message commands, defaults to `cmd_vel` -1-> -->
-    <!--   <command_topic>/jetauto/cmd_vel</command_topic> -->
-    <!--     <!-1- Topic to publish nav_msgs/Odometry messages, defaults to `odom` -1-> -->
-    <!--   <odometry_topic>jetauto/odom/unfiltered</odometry_topic> -->
-    <!--     <!-1- Odometry frame, defaults to `odom` -1-> -->
-    <!--   <odometry_frame>odom</odometry_frame> -->
-    <!--     <!-1- Robot frame to calculate odometry from, defaults to `base_footprint` -1-> -->
-    <!--   <robot_base_frame>base_footprint</robot_base_frame> -->
-    <!--     <!-1- Odometry source, 0 for ENCODER, 1 for WORLD, defaults to WORLD -1-> -->
-    <!--   <odometry_source>0</odometry_source> -->
-    <!--     <!-1- Set to true to publish transforms for the wheel links, defaults to false -1-> -->
-    <!--   <publish_wheel_tF>false</publish_wheel_tF> -->
-    <!--     <!-1- Set to true to publish transforms for the odometry, defaults to true -1-> -->
-    <!--   <publish_odom>false</publish_odom> -->
-    <!--     <!-1- Set to true to publish sensor_msgs/JointState on /joint_states for the wheel joints, defaults to false -1-> -->
-    <!--   <publish_wheel_joint_state>false</publish_wheel_joint_state> -->
-    <!--     <!-1- Set to true to swap right and left wheels, defaults to true -1-> -->
-    <!--   <legacy_mode>false</legacy_mode> -->
-    <!-- </plugin> -->
-  </gazebo>
-  <!-- Transmission macro -->
-  <!-- <xacro:macro name="SimpleTransmissionPosition" params="joint"> -->
-  <!--     <transmission name="tran_${joint}"> -->
-  <!--         <type>transmission_interface/SimpleTransmission</type> -->
-  <!--         <joint name="${joint}"> -->
-  <!--             <hardwareInterface>hardware_interface/PositionJointInterface</hardwareInterface> -->
-  <!--         </joint> -->
-  <!--         <actuator name="${joint}_motor"> -->
-  <!--             <hardwareInterface>hardware_interface/PositionJointInterface</hardwareInterface> -->
-  <!--             <mechanicalReduction>1</mechanicalReduction> -->
-  <!--         </actuator> -->
-  <!--     </transmission> -->
-  <!-- </xacro:macro> -->
-  <!-- <xacro:SimpleTransmissionPosition joint="joint1" /> -->
-</robot>
+/home/jose/Documents/robotica/src/robotics_class/urdf/jetauto_car.urdf.xacro
