Commit message: feat: update params and launch file

File: install/robotics_class/share/robotics_class/urdf/lidar.urdf.xacro (robot description, xacro)
@@ -1,92 +1 @@
-<?xml version="1.0" encoding="utf-8"?>
-<robot name="lidar" xmlns:xacro="http://ros.org/wiki/xacro" >
-  <xacro:property name="M_PI" value="3.1415926535897931"/>
-  <link
-    name="lidar_link">
-    <inertial>
-      <origin
-        xyz="-0.0157049024536227 0.000340793431659825 -0.0214732100882973"
-        rpy="0 0 0" />
-      <mass
-        value="0.0522535578752524" />
-      <inertia
-        ixx="1.4542908499666E-05"
-        ixy="4.8193721668021E-08"
-        ixz="2.30575406031324E-07"
-        iyy="1.85618648837978E-05"
-        iyz="-1.29750110413905E-08"
-        izz="3.10574357987674E-05" />
-    </inertial>
-    <visual>
-      <origin
-        xyz="0 0 0"
-        rpy="0 0 0" />
-      <geometry>
-        <mesh
-          filename="package://robotics_class/models/jetauto/lidar_link.stl" />
-      </geometry>
-      <material name="black"/>
-    </visual>
-    <!--<collision>-->
-      <!--<origin-->
-        <!--xyz="0 0 0"-->
-        <!--rpy="0 0 0" />-->
-      <!--<geometry>-->
-        <!--<mesh-->
-          <!--filename="package://robotics_class/models/jetauto/lidar_link.stl" />-->
-      <!--</geometry>-->
-    <!--</collision>-->
-  </link>
-  <joint
-    name="lidar_joint"
-    type="fixed">
-    <origin
-      xyz="0.0959394346777203 -1.03974386779226E-05 0.128396206697751"
-      rpy="0 0 0" />
-    <parent
-      link="base_link" />
-    <child
-      link="lidar_link" />
-    <axis
-      xyz="0 0 0" />
-  </joint>
-  <gazebo reference="lidar_link">
-    <sensor name="lidar" type="ray">
-      <always_on>true</always_on>
-      <update_rate>10</update_rate>
-      <visualize>false</visualize>
-      <ray>
-        <scan>
-          <horizontal>
-            <!-- <xacro:if value="${optionals['use_less_scan_samples']}"> -->
-            <samples>180</samples>
-            <!-- </xacro:if> -->
-            <!-- <xacro:unless value="${optionals['use_less_scan_samples']}"> -->
-            <!--   <samples>${16000/15}</samples> -->
-            <!-- </xacro:unless> -->
-            <resolution>1</resolution>
-            <min_angle>-2.3562</min_angle>
-            <max_angle>2.3562</max_angle>
-          </horizontal>
-        </scan>
-        <range>
-          <min>0.15</min>
-          <max>11</max>
-          <resolution>0.01</resolution>
-        </range>
-        <noise>
-          <type>gaussian</type>
-          <mean>0.0</mean>
-          <stddev>0.01</stddev>
-        </noise>
-      </ray>
-      <plugin name="gazebo_ros_ray_sensor" filename="libgazebo_ros_ray_sensor.so">
-        <ros>
-          <remapping>~/out:=/jetauto/lidar/scan</remapping>
-        </ros>
-        <frame_name>lidar_link</frame_name>
-        <output_type>sensor_msgs/LaserScan</output_type>
-      </plugin>
-    </sensor>
-  </gazebo>
-</robot>
+/home/jose/Documents/robotica/src/robotics_class/urdf/lidar.urdf.xacro

File: install/robotics_class/share/robotics_class/urdf/materials.xacro (robot description, xacro)
@@ -1,27 +1 @@
-<?xml version="1.0"?>
-<robot>
-    <material name="black">
-        <color rgba="0.1 0.1 0.1 1.0"/>
-    </material>
-    <material name="blue">
-        <color rgba="0.0 0.0 0.8 1.0"/>
-    </material>
-    <material name="green">
-        <color rgba="0.4 0.9 0.4 1.0"/>
-    </material>
-    <material name="gray">
-        <color rgba="0.7 0.7 0.7 1.0"/>
-    </material>
-    <material name="darkgray">
-        <color rgba="0.3 0.3 0.3 1.0"/>
-    </material>
-    <material name="red">
-        <color rgba="0.8 0.0 0.0 1.0"/>
-    </material>
-    <material name="white">
-        <color rgba="1.0 1.0 1.0 1.0"/>
-    </material>
-    <material name="yellow">
-        <color rgba="0.8 0.8 0.0 1.0"/>
-    </material>
-</robot>
+/home/jose/Documents/robotica/src/robotics_class/urdf/materials.xacro

File: install/robotics_class/share/robotics_class/urdf/p3d_plugin.gazebo.xacro (robot description, xacro)
@@ -1,29 +1 @@
-<?xml version="1.0"?>
-<robot xmlns:xacro="http://ros.org/wiki/xacro">
-  <xacro:macro name="p3d_plugin_macro" params="parent update_rate topic_name mass body_name frame_name noise xyz_offset rpy_offset *inertia *origin">
-    <link name="odometry_ground_truth_link">
-      <xacro:insert_block name="inertia"/>
-      <mass value="${mass}"/>
-    </link>
-    <joint name="odometry_ground_truth_link_joint" type="revolute">
-      <parent link="${parent}"/>
-      <xacro:insert_block name="origin"/>
-      <child link="odometry_ground_truth_link"/>
-      <limit upper="0" lower="0" effort="0" velocity="0"/>
-    </joint>
-    <gazebo>
-      <plugin name="gazebo_ros_p3d" filename="libgazebo_ros_p3d.so">
-        <ros>
-          <remapping>odom:=odometry/ground_truth</remapping>
-        </ros>
-        <always_on>true</always_on>
-        <update_rate>${update_rate}</update_rate>
-        <body_name>${body_name}</body_name>
-        <gaussian_noise>${noise}</gaussian_noise>
-        <frame_name>${frame_name}</frame_name>
-        <xyz_offset>${xyz_offset}</xyz_offset>
-        <rpy_offset>${rpy_offset}</rpy_offset>
-      </plugin>
-    </gazebo>
-  </xacro:macro>
-</robot>
+/home/jose/Documents/robotica/src/robotics_class/urdf/p3d_plugin.gazebo.xacro
